File: nano_samc21e.kicad_pcb (KiCad board)
At the start: 2 copper layers, 17.9 x 38.2 mm, 35 parts, among them J1 SWD, J2 Castellated_headers, SW1 RST, U1 ATSAMC21E18A-M, U2 AP2112K-3.3, U3 LMZM23600V5, Y1 32.768kHz 12.5p

Commit message: Added missing pin numbering Added WEEE logo Added JLCPCB order number Generated fresh JLCPCB output files
Parts:
- added ?: , clipboard:e8e54784-63be-4e29-bba0-8d06d3e6b108, B.Cu at (48.0, 42.0)
- added FID6: WEEE, Symbol:WEEE-Logo_4.2x6mm_SilkScreen, B.Cu at (24.4, 49.1)
Other:
- board text added: "JLCJLCJLCJLC"
